Commit message: Update mypalletizer_260_m5.urdf

File: MyPalletizer260_gazebo/config/mypalletizer_260_m5.urdf (robot description, URDF)
Before this commit: robot firefighter, 14 links, 13 joints
Joints:
- removed joint joint4_to_joint3
- added joint joint4_to_joint3_fixed: type fixed, parent link3, child link4, origin xyz=0.134 -0.005   0.0 rpy=3.1415926 0 0 
- joint joint3_to_joint2: limit lower=-1.6057 upper=1.0471 effort=1000.0 velocity=1 -> lower=-0.96 upper=0.96 effort=1000.0 velocity=1
- joint joint5_to_joint4: limit lower=-3.14 upper=3.14 effort=1000.0 velocity=1 -> lower=-2.53 upper=2.53 effort=1000.0 velocity=1
